File: my_arduino_frankenstein/my_arduino_frankenstein.kicad_sch (KiCad schematic)
At the start: 7 parts, among them U1 LM358

Commit message: progress 2
Parts:
- added C10, C11, C12, C5, C6, C7, C8, C9: C, symbol Device:C
- added D2: D, symbol Device:D
- added U2: NCP115AMX250TCG, Package_DFN_QFN:OnSemi_XDFN4-1EP_1.0x1.0mm_EP0.52x0.52mm, symbol Regulator_Linear:NCP115AMX250TCG
- added U3: CH340G, Package_SO:SOIC-16_3.9x9.9mm_P1.27mm, symbol Interface_USB:CH340G
Connections:
- net GND: now also C1.2, U2.2 (GND), U2.3 (EN), U2.4 (IN), U2.5 (GND)
- net at C1.1: now also D2.1 (K), U2.1 (OUT)
Other:
- moved on the sheet: C1

Commit message: progress 3
Parts:
- added R14_10k, R15_10k: R, symbol Device:R
- added U4: TSV994, symbol Amplifier_Operational:TSV994
- added U5: ATmega328P-M, Package_DFN_QFN:QFN-32-1EP_5x5mm_P0.5mm_EP3.1x3.1mm, symbol MCU_Microchip_ATmega:ATmega328P-M
- renumbered C1 to 47u25v
Connections:
- net GND: now also R15_10k.2
- net at 47u25v.1, D2.1 (K), U2.1 (OUT): now also R14_10k.1
- new net: U5.21 (GND), U5.3 (GND), U5.33 (GND), U5.5 (GND)
- new net: U5.4 (VCC), U5.6 (VCC)
- new net: R14_10k.2, R15_10k.1, U4.3 (+)

Commit message: progress 5
Parts:
- removed C11, C12, C7, C8, C9: C, symbol Device:C
- removed D1: LED, symbol Device:LED
- added C1, C5, C6: C, symbol Device:C
- added C14, C16: 100n, symbol Device:C
- added C20, C21: 22p, symbol Device:C
- added D1: D, symbol Device:D
- added D2, D3: ON, symbol Device:LED_Filled
- added J1, J2, J3: Conn_01x09_Pin, symbol Connector:Conn_01x09_Pin
- added R: 1M, symbol Device:R
- added R13: 10k, symbol Device:R
- added R17, R6, R7, R8, R9: 1k, symbol Device:R
- added RX, TX: LED, symbol Device:LED
- added S1: RESET, EVQ-PF008K:RIGHTANGLE-PUSHBUTTON, symbol EVQ-PF008K:EVQ-PF008K
- added U7: LM358M, LM358M:SOIC127P599X175-8N, symbol LM358M:LM358M
- added Y: 12Mhz, symbol Device:Crystal
- added Z1: 16Mhz, symbol Device:Crystal
- C: renamed from 47u25v; value C -> 47u25v
- C11: renamed from C3; value C -> 100n
- C13: renamed from C5; value C -> 100n
- C15: renamed from C6; value C -> 100n
- C2: value C -> 47u 25V
- C4: value C -> 100n
- R14: renamed from R14_10k; value R -> 10k
- R15: renamed from R15_10k; value R -> 10k
- R4: renamed from R1; value R -> 1k
- renumbered D2 to VD
Connections:
- net GND: now also C13.2, C15.2, U3.1 (GND), U5.21 (GND), U5.3 (GND), U5.33 (GND), U5.5 (GND), C14.1, C16.1, C20.2, C21.2, C5.2, C6.2, D2.2 (A), D3.2 (A), S1.A, U7.4 (GND); no longer C11.1, C2.1, C4.1, U2.3 (EN), U2.4 (IN)
- net +5V: now reaches C10.1
- net +5V: now also C11.1, C13.1, C2.1, C4.1, U2.3 (EN), U2.4 (IN), U3.16 (VCC), U5.18 (AVCC), U5.4 (VCC), U5.6 (VCC), C14.2, D1.1 (K), R13.1, R13.2, R17.2, R6.2, R7.2, S1.B
- net at C10.2: now also U3.4 (V3)
- net at U5.16 (PB4): now also U1.3 (+)
- net at U5.20 (AREF): now also C16.2
- net at U5.29 (~{RESET}/PC6): now also C1.2
- net at U5.30 (PD0): now also R8.2, TX.1 (K)
- net at U5.31 (PD1): now also R9.2, RX.1 (K)
- net at U5.7 (XTAL1/PB6): now also C5.1, R.1, Z1.2
- net at U5.8 (XTAL2/PB7): now also C6.1, R.2, Z1.1
- net at U4.2 (-): now also C15.1
- net at R4.2: now also D3.1 (K)
- net at U3.13 (~{DTR}): now also C1.1
- net at U3.2 (TXD): now also R8.1
- net at U3.3 (RXD): now also R9.1
- net at U3.5 (UD+): now also U7.3 (POSA)
- net at U3.6 (UD-): now also U7.2 (NEGA)
- net at U3.7 (XI): now also C20.1, Y.1
- net at U3.8 (XO): now also C21.1, Y.2
- new net: R6.1, RX.2 (A)
- new net: R7.1, TX.2 (A)
- new net: D2.1 (K), R17.1
Other:
- moved on the sheet: C, C10, C11, C13, C15, C2, C4, R14, R15, R4, U2, U4A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

Commit message: progress 6
Parts:
- removed J1, J2, J3: Conn_01x09_Pin, symbol Connector:Conn_01x09_Pin
- added AD: 6X1F-H8,5, symbol Connector:Conn_01x06_Pin
- added IOH: 10X1F-H8,5, symbol Connector:Conn_01x10_Socket
- added IOL, POWER: 8X1F-H8,5, symbol Connector:Conn_01x08_Socket
- added J1: Conn_02x03_Odd_Even, symbol Connector_Generic:Conn_02x03_Odd_Even
- added J4, J5, J7: Conn_01x04_Pin, symbol Connector:Conn_01x04_Pin
- added PT1: L, symbol Device:L
Connections:
- net +5V: now also J1.2 (Pin_2), J1.5 (Pin_5), J4.3 (Pin_3), J5.2 (Pin_2), J7.3 (Pin_3), POWER.2 (Pin_2), POWER.5 (Pin_5)
- net GND: now also IOH.7 (Pin_7), J1.6 (Pin_6), J4.4 (Pin_4), J5.1 (Pin_1), J7.4 (Pin_4), POWER.6 (Pin_6), POWER.7 (Pin_7)
- net at R9.2, RX.1 (K), U5.31 (PD1): now also IOL.2 (Pin_2)
- net at C.1, R14.1, U2.1 (OUT)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: now also POWER.8 (Pin_8)
- net at U5.1 (PD3): now also IOL.4 (Pin_4)
- net at U5.10 (PD6): now also IOL.7 (Pin_7)
- net at U5.11 (PD7): now also IOL.8 (Pin_8)
- net at U5.12 (PB0): now also IOH.1 (Pin_1)
- net at U5.13 (PB1): now also IOH.2 (Pin_2)
- net at U5.14 (PB2): now also IOH.3 (Pin_3)
- net at U5.15 (PB3): now also IOH.4 (Pin_4), J1.4 (Pin_4)
- net at U1.3 (+), U5.16 (PB4): now also IOH.5 (Pin_5), J1.3 (Pin_3)
- net at U5.17 (PB5): now also IOH.6 (Pin_6), J1.1 (Pin_1)
- net at U5.2 (PD4): now also IOL.5 (Pin_5)
- net at C16.2, U5.20 (AREF): now also IOH.8 (Pin_8)
- net at U5.23 (PC0): now also AD.6 (Pin_6)
- net at U5.24 (PC1): now also AD.5 (Pin_5)
- net at U5.25 (PC2): now also AD.4 (Pin_4)
- net at U5.26 (PC3): now also AD.3 (Pin_3)
- net at U5.27 (PC4): now also AD.2 (Pin_2), IOH.9 (Pin_9), J7.2 (Pin_2)
- net at U5.28 (PC5): now also AD.1 (Pin_1), IOH.10 (Pin_10), J7.1 (Pin_1)
- net at C1.2, U5.29 (~{RESET}/PC6): now also POWER.3 (Pin_3)
- net at R8.2, TX.1 (K), U5.30 (PD0): now also IOL.1 (Pin_1)
- net at U5.32 (PD2): now also IOL.3 (Pin_3)
- net at U5.9 (PD5): now also IOL.6 (Pin_6)
- net at C15.1, U4.2 (-): now also J5.3 (Pin_3), J5.4 (Pin_4), POWER.4 (Pin_4)
- net at U7.8 (V+): now also PT1.2
- net at D1.2 (A): now also PT1.1
Other:
- moved on the sheet: C14, C5, C6

Commit message: final schematics for compact board
Parts:
- removed AD: 6X1F-H8,5, symbol Connector:Conn_01x06_Pin
- removed C: 47u25v, symbol Device:C
- removed C11, C13, C15, C4: 100n, symbol Device:C
- removed C2: 47u 25V, symbol Device:C
- removed D1, VD: D, symbol Device:D
- removed D3: ON, symbol Device:LED_Filled
- removed J4, J5, J7: Conn_01x04_Pin, symbol Connector:Conn_01x04_Pin
- removed PT1: L, symbol Device:L
- removed R14, R15: 10k, symbol Device:R
- removed R6, R7, R8, R9: 1k, symbol Device:R
- removed RX, TX: LED, symbol Device:LED
- removed S1: RESET, EVQ-PF008K:RIGHTANGLE-PUSHBUTTON, symbol EVQ-PF008K:EVQ-PF008K
- removed U1: LM358, symbol Amplifier_Operational:LM358
- removed U2: NCP115AMX250TCG, Package_DFN_QFN:OnSemi_XDFN4-1EP_1.0x1.0mm_EP0.52x0.52mm, symbol Regulator_Linear:NCP115AMX250TCG
- removed U4: TSV994, symbol Amplifier_Operational:TSV994
- removed U7: LM358M, LM358M:SOIC127P599X175-8N, symbol LM358M:LM358M
- added AD1: 6X1F-H8,5, Connector_PinSocket_1.27mm:PinSocket_1x06_P1.27mm_Vertical, symbol Connector:Conn_01x06_Socket
- added J2: USB3_A, Connector_USB:USB3_A_Molex_48393-001, symbol Connector:USB3_A
- added R2, R3, R5: 1k, Resistor_SMD:R_0201_0603Metric, symbol Device:R
- added RX1, TX1: LED, LED_SMD:LED-APA102-2020, symbol Device:LED
- added SW1: SW_DIP_x01, Button_Switch_SMD:Nidec_Copal_CAS-120A, symbol Switch:SW_DIP_x01
- C1, C10, C14, C16, C20, C21, C5, C6: footprint (none) -> Capacitor_SMD:CP_Elec_3x5.3
- D2: footprint (none) -> LED_SMD:LED-APA102-2020
- IOH1: renamed from IOH; footprint (none) -> Connector_PinSocket_1.27mm:PinSocket_1x10_P1.27mm_Vertical
- IOL1: renamed from IOL; footprint (none) -> Connector_PinHeader_2.54mm:PinHeader_1x08_P2.54mm_Vertical
- J1: footprint (none) -> Connector_PinHeader_2.00mm:PinHeader_2x03_P2.00mm_Vertical
- POWER1: renamed from POWER; footprint (none) -> Connector_PinSocket_2.00mm:PinSocket_1x08_P2.00mm_Vertical
- R1: renamed from R; footprint (none) -> Resistor_SMD:R_0201_0603Metric
- R13, R17, R4: footprint (none) -> Resistor_SMD:R_0201_0603Metric
- Y1: renamed from Y; footprint (none) -> Crystal:Crystal_AT310_D3.0mm_L10.0mm_Horizontal
- Z1: footprint (none) -> Crystal:Crystal_AT310_D3.0mm_L10.0mm_Horizontal
Connections:
- net GND is gone; now on net +5V: C14.1, C16.1, C20.2, C21.2, C5.2, C6.2, D2.2 (A), IOH1.7 (Pin_7), J1.6 (Pin_6), POWER1.6 (Pin_6), POWER1.7 (Pin_7), U3.1 (GND), U5.21 (GND), U5.3 (GND), U5.33 (GND), U5.5 (GND)
- net +5V: now also IOH1.4 (Pin_4), IOH1.5 (Pin_5), J1.3 (Pin_3), J1.4 (Pin_4), POWER1.8 (Pin_8), U5.15 (PB3), U5.16 (PB4), J2.4 (GND), R3.2, R5.2, SW1.1, SW1.2
- net at IOL1.2 (Pin_2), U5.31 (PD1): now also R4.2, RX1.1 (K)
- net at IOL1.1 (Pin_1), U5.30 (PD0): now also R2.2, TX1.1 (K)
- net at IOH1.10 (Pin_10), U5.28 (PC5): now also AD1.6 (Pin_6)
- net at IOH1.9 (Pin_9), U5.27 (PC4): now also AD1.5 (Pin_5)
- net at U5.23 (PC0): now also AD1.1 (Pin_1)
- net at U5.24 (PC1): now also AD1.2 (Pin_2)
- net at U5.25 (PC2): now also AD1.3 (Pin_3)
- net at U5.26 (PC3): now also AD1.4 (Pin_4)
- net at U3.6 (UD-): now also J2.2 (D-)
- net at U3.5 (UD+): now also J2.3 (D+)
- net at U3.3 (RXD): now also R4.1
- net at U3.2 (TXD): now also R2.1
- new net: R5.1, RX1.2 (A)
- new net: R3.1, TX1.2 (A)
Other:
- moved on the sheet: C10, C14, C16, C20, C21, C5, C6, IOH1, IOL1, POWER1, R1, R13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
